Commit message: added inertia tags

File: src/axlr_description/urdf/axlr_core.urdf.xacro (robot description, xacro)
@@ -1,21 +1,3 @@
 <robot xmlns:xacro="http://www.ros.org/wiki/xacro">
-    <xacro:property name="base_length" value="0.266"/>
-    <xacro:property name="base_width" value="0.237"/>
-    <xacro:property name="base_height" value="0.122"/>
-    <xacro:property name="wheel_offset_from_ground" value="0.072"/>
-    <xacro:property name="wheel_offset_from_width" value="0.0325"/>
-    <xacro:property name="wheel_offset_from_side" value="0.025"/>
-    <xacro:property name="wheel_offset_from_top" value="0.03"/>
-    <xacro:property name="caster_wheel_radius" value="0.015"/>
-    <xacro:property name="caster_wheel_offset_from_top" value="0.03"/>
-    <xacro:property name="wheel_diameter" value="0.084"/>
-    <xacro:property name="wheel_length" value="0.04"/>
-    <xacro:property name="PI" value="3.14159"/>
-    <material name="white">
-        <color rgba="1.0 1.0 1.0 1.0"/>
-    </material>
-    <material name="black">
-        <color rgba="0.0 0.0 0.0 1.0"/>
-    </material>
     <link name="world">
     </link>
@@ -35,4 +17,6 @@
             <material name="white"/>
         </collision>
+        <xacro:box_inertia  m="2.5" l="${base_length}" w="${base_width}" h="${base_height}"
+            xyz="0.0 ${-wheel_offset_from_width} ${base_height/2}" rpy="0.0 0.0 0.0"/>
     </link>
     <joint name="world_base" type="fixed">
@@ -56,4 +40,6 @@
             <material name="black"/>
         </collision>
+        <xacro:cylinder_inertia m="0.1" r="${wheel_diameter/2}" h="${wheel_length}"
+                xyz="0.0 0.0 0.0" rpy="0.0 0.0 0.0"/>
     </link>
     <joint name="base_right_wheel" type="continuous">
@@ -78,4 +64,6 @@
             <material name="black"/>
         </collision>
+        <xacro:cylinder_inertia m="0.1" r="${wheel_diameter/2}" h="${wheel_length}"
+                xyz="0.0 0.0 0.0" rpy="0.0 0.0 0.0"/>
     </link>
     <joint name="base_left_wheel" type="continuous">
@@ -100,4 +88,6 @@
             <material name="black"/>
         </collision>
+        <xacro:box_inertia  m="0.2" l="0.02" w="0.02" h="0.06"
+                xyz="0.0 0.0 -0.03" rpy="0.0 0.0 0.0"/>
     </link>
     <joint name="base_back_support" type="fixed">
@@ -121,4 +111,6 @@
             <material name="white"/>
         </collision>
+        <xacro:sphere_inertia m="0.2" r="${caster_wheel_radius}"
+                xyz="0.0 0.0 0.0" rpy="0.0 0.0 0.0"/>
     </link>
     <joint name="base_caster_wheel" type="fixed">

File: src/axlr_description/urdf/main.urdf.xacro (robot description, xacro)
@@ -1,3 +1,5 @@
 <robot xmlns:xacro="http://www.ros.org/wiki/xacro" name="AXLR">
+    <xacro:include filename="properties.urdf.xacro"/>
+    <xacro:include filename="inertial_macros.urdf.xacro"/>
     <xacro:include filename="axlr_core.urdf.xacro"/>
 </robot>

Commit message: have not successfully fixed simulation

File: src/axlr_description/urdf/axlr_core.urdf.xacro (robot description, xacro)
@@ -1,5 +1,5 @@
+<?xml version="1.0"?>
 <robot xmlns:xacro="http://www.ros.org/wiki/xacro">
-    <link name="world">
-    </link>
+    <link name="world"/>
     <link name="base_link">
         <visual>
@@ -23,5 +23,5 @@
         <parent link="world"/>
         <child link="base_link"/>
-        <origin xyz="0.0 ${wheel_offset_from_width} ${wheel_offset_from_ground}" rpy="0.0 0.0 0.0"/>
+        <origin xyz="0.0 ${wheel_offset_from_width} ${wheel_offset_from_ground}" rpy="0.0 0.0 ${-PI/2}"/>
     </joint>
     <link name="right_wheel">

File: src/axlr_description/urdf/inertial_macros.urdf.xacro (robot description, xacro)
@@ -1,2 +1,3 @@
+<?xml version="1.0"?>
 <robot xmlns:xacro="http://www.ros.org/wiki/xacro">
     <xacro:macro name = "box_inertia" params="m l w h xyz rpy">

File: src/axlr_description/urdf/main.urdf.xacro (robot description, xacro)
@@ -1,5 +1,8 @@
+<?xml version="1.0"?>
 <robot xmlns:xacro="http://www.ros.org/wiki/xacro" name="AXLR">
     <xacro:include filename="properties.urdf.xacro"/>
     <xacro:include filename="inertial_macros.urdf.xacro"/>
     <xacro:include filename="axlr_core.urdf.xacro"/>
+    <xacro:include filename="gazebo_properties.urdf.xacro"/>
+    <xacro:include filename="axlr_ros2_control.urdf.xacro"/>
 </robot>

File: src/axlr_description/urdf/properties.urdf.xacro (robot description, xacro)
@@ -1,2 +1,3 @@
+<?xml version="1.0"?>
 <robot xmlns:xacro="http://www.ros.org/wiki/xacro">
     <xacro:property name="base_length" value="0.266"/>
@@ -12,4 +13,5 @@
     <xacro:property name="wheel_length" value="0.04"/>
     <xacro:property name="PI" value="3.14159"/>
+    <xacro:property name="wheel_seperation" value="0.316"/>
     <material name="white">
         <color rgba="1.0 1.0 1.0 1.0"/>

Commit message: started the urdf again

File: src/axlr_description/urdf/axlr_core.urdf.xacro (robot description, xacro)
@@ -4,26 +4,26 @@
     <link name="base_link">
         <visual>
-            <origin xyz="0.0 ${-wheel_offset_from_width} ${base_height/2}" rpy="0.0 0.0 0.0"/>
+            <origin xyz="${-center_offset} 0.0 ${base_height/2}" rpy="0.0 0.0 0.0"/>
             <geometry>
-                <box size="${base_length} ${base_width} ${base_height}"/>
+                <box size="${base_width} ${base_length} ${base_height}"/>
             </geometry>
             <material name="white"/>
         </visual>
         <collision>
-            <origin xyz="0.0 ${-wheel_offset_from_width} ${base_height/2}" rpy="0.0 0.0 0.0"/>
+            <origin xyz="${-center_offset} 0.0 ${base_height/2}" rpy="0.0 0.0 0.0"/>
             <geometry>
-                <box size="${base_length} ${base_width} ${base_height}"/>
+                <box size="${base_width} ${base_length} ${base_height}"/>
             </geometry>
             <material name="white"/>
         </collision>
-        <xacro:box_inertia  m="2.5" l="${base_length}" w="${base_width}" h="${base_height}"
-            xyz="0.0 ${-wheel_offset_from_width} ${base_height/2}" rpy="0.0 0.0 0.0"/>
+        <xacro:box_inertia m="1.0" l="${base_width}" w="${base_length}" h="${base_height}"
+                xyz="${-center_offset} 0.0 ${base_height/2}" rpy="0.0 0.0 0.0"/>
     </link>
-    <joint name="world_base" type="fixed">
+    <joint name="world_joint" type="fixed">
         <parent link="world"/>
         <child link="base_link"/>
-        <origin xyz="0.0 ${wheel_offset_from_width} ${wheel_offset_from_ground}" rpy="0.0 0.0 ${-PI/2}"/>
+        <origin xyz="${center_offset} 0.0 ${wheel_diameter/2}" rpy="0.0 0.0 0.0"/>
     </joint>
-    <link name="right_wheel">
+    <link name="right_wheel_link">
         <visual>
             <origin xyz="0.0 0.0 0.0" rpy="0.0 0.0 0.0"/>
@@ -40,14 +40,14 @@
             <material name="black"/>
         </collision>
-        <xacro:cylinder_inertia m="0.1" r="${wheel_diameter/2}" h="${wheel_length}"
-                xyz="0.0 0.0 0.0" rpy="0.0 0.0 0.0"/>
+        <xacro:cylinder_inertia m="0.5" r ="${wheel_diameter/2}" h="${wheel_length}"
+             xyz="0.0 0.0 0.0" rpy="0.0 0.0 0.0"/>
     </link>
-    <joint name="base_right_wheel" type="continuous">
+    <joint name="right_wheel_joint" type="continuous">
+        <origin xyz="0.0 -${base_length/2 + wheel_offset_from_side} 0.0" rpy="${PI/2} 0.0 0.0"/>
         <parent link="base_link"/>
-        <child link="right_wheel"/>
-        <origin xyz="${base_length/2+wheel_offset_from_side} 0.0 ${-wheel_offset_from_top}" rpy="0.0 ${PI/2} 0.0"/>
-        <axis xyz="0.0 0.0 1.0"/>
+        <child link="right_wheel_link"/>
+        <axis xyz="0.0 0.0 -1.0"/>
     </joint>
-    <link name="left_wheel">
+    <link name="left_wheel_link">
         <visual>
             <origin xyz="0.0 0.0 0.0" rpy="0.0 0.0 0.0"/>
@@ -64,58 +64,33 @@
             <material name="black"/>
         </collision>
-        <xacro:cylinder_inertia m="0.1" r="${wheel_diameter/2}" h="${wheel_length}"
-                xyz="0.0 0.0 0.0" rpy="0.0 0.0 0.0"/>
+        <xacro:cylinder_inertia m="0.5" r ="${wheel_diameter/2}" h="${wheel_length}"
+             xyz="0.0 0.0 0.0" rpy="0.0 0.0 0.0"/>
     </link>
-    <joint name="base_left_wheel" type="continuous">
+    <joint name="left_wheel_joint" type="continuous">
+        <origin xyz="0.0 ${base_length/2 + wheel_offset_from_side} 0.0" rpy="${PI/2} 0.0 0.0"/>
         <parent link="base_link"/>
-        <child link="left_wheel"/>
-        <origin xyz="-${base_length/2+wheel_offset_from_side} 0.0 ${-wheel_offset_from_top}" rpy="0.0 ${-PI/2} 0.0"/>
-        <axis xyz="0.0 0.0 1.0"/>
+        <child link="left_wheel_link"/>
+        <axis xyz="0.0 0.0 -1.0"/>
     </joint>
-    <link name="back_support">
+    <link name="caster_wheel_link">
         <visual>
-            <origin xyz="0.0 0.0 -0.03" rpy="0.0 0.0 0.0"/>
+            <origin xyz="0.0 0.0 0.0" rpy="0.0 0.0 0.0"/>
             <geometry>
-                <box size="0.02 0.02 0.06"/>
+                <sphere radius="${wheel_diameter/4}"/>
             </geometry>
             <material name="black"/>
         </visual>
         <collision>
-            <origin xyz="0.0 0.0 -0.03" rpy="0.0 0.0 0.0"/>
+            <origin xyz="0.0 0.0 0.0" rpy="0.0 0.0 0.0"/>
             <geometry>
-                <box size="0.02 0.02 -0.06"/>
+                <sphere radius="${wheel_diameter/4}"/>
             </geometry>
             <material name="black"/>
         </collision>
-        <xacro:box_inertia  m="0.2" l="0.02" w="0.02" h="0.06"
-                xyz="0.0 0.0 -0.03" rpy="0.0 0.0 0.0"/>
     </link>
-    <joint name="base_back_support" type="fixed">
+    <joint name="caster_joint" type="fixed">
+        <origin xyz="-${base_width/2} 0.0 -${wheel_diameter/4}" rpy="0.0 0.0 0.0"/>
         <parent link="base_link"/>
-        <child link="back_support"/>
-        <origin xyz="0.0 -${base_width/2+wheel_offset_from_width-0.02} 0.0" rpy="0.0 0.0 0.0"/>
-    </joint>
-    <link name="base_caster_wheel">
-        <visual>
-            <origin xyz="0.0 0.0 0.0" rpy="0.0 0.0 0.0"/>
-            <geometry>
-                    <sphere radius="${caster_wheel_radius}"/>
-            </geometry>
-            <material name="white"/>
-        </visual>
-        <collision>
-            <origin xyz="0.0 0.0 0.0" rpy="0.0 0.0 0.0"/>
-            <geometry>
-                    <sphere radius="${caster_wheel_radius}"/>
-            </geometry>
-            <material name="white"/>
-        </collision>
-        <xacro:sphere_inertia m="0.2" r="${caster_wheel_radius}"
-                xyz="0.0 0.0 0.0" rpy="0.0 0.0 0.0"/>
-    </link>
-    <joint name="base_caster_wheel" type="fixed">
-        <parent link="back_support"/>
-        <child link="base_caster_wheel"/>
-        <origin xyz="0.0 0.0 -0.06" rpy="0.0 0.0 0.0"/>
+        <child link="caster_wheel_link"/>
     </joint>
 </robot>

File: src/axlr_description/urdf/properties.urdf.xacro (robot description, xacro)
@@ -8,8 +8,8 @@
     <xacro:property name="wheel_offset_from_side" value="0.025"/>
     <xacro:property name="wheel_offset_from_top" value="0.03"/>
-    <xacro:property name="caster_wheel_radius" value="0.015"/>
-    <xacro:property name="caster_wheel_offset_from_top" value="0.03"/>
     <xacro:property name="wheel_diameter" value="0.084"/>
     <xacro:property name="wheel_length" value="0.04"/>
+    <xacro:property name="center_offset" value="0.0285"/>
+    <xacro:property name="caster_offset" value="0.0285"/>
     <xacro:property name="PI" value="3.14159"/>
     <xacro:property name="wheel_seperation" value="0.316"/>

Commit message: still nothing

File: src/axlr_description/urdf/axlr_core.urdf.xacro (robot description, xacro)
@@ -88,4 +88,6 @@
             <material name="black"/>
         </collision>
+        <xacro:sphere_inertia m="0.5" r ="${wheel_diameter/4}"
+                xyz="0.0 0.0 0.0" rpy="0.0 0.0 0.0"/>
     </link>
     <joint name="caster_joint" type="fixed">

File: src/axlr_description/urdf/axlr_ros2_control.urdf.xacro (robot description, xacro)
@@ -5,5 +5,5 @@
             <plugin>gazebo_ros2_control/GazeboSystem</plugin>
         </hardware>
-        <joint name="base_right_wheel">
+        <joint name="right_wheel_joint">
             <command_interface name="velocity">
                 <param name="min">-10</param>
@@ -13,5 +13,5 @@
             <state_interface name="velocity"/>
         </joint>
-        <joint name="base_left_wheel">
+        <joint name="left_wheel_joint">
             <command_interface name="velocity">
                 <param name="min">-10</param>

File: src/axlr_description/urdf/gazebo_properties.urdf.xacro (robot description, xacro)
@@ -3,5 +3,5 @@
     <transmission name="right_wheel_transmission">
         <actuator name="right_wheel_motor" role="right_wheel_actuator"/>
-        <joint name="base_right_wheel" role="right_joint">
+        <joint name="right_wheel_joint" role="right_joint">
             <mechanicalReduction>1.0</mechanicalReduction>
         </joint>
@@ -10,5 +10,5 @@
     <transmission name="left_wheel_transmission">
         <actuator name="left_wheel_motor" role="left_wheel_actuator"/>
-        <joint name="base_left_wheel" role="left_joint">
+        <joint name="left_wheel_joint" role="left_joint">
             <mechanicalReduction>1.0</mechanicalReduction>
         </joint>
@@ -18,32 +18,14 @@
         <material>Gazebo/White</material>
     </gazebo>
-    <gazebo reference="right_wheel">
+    <gazebo reference="right_wheel_link">
         <material>Gazebo/Black</material>
-        <mu1>100000000000000.0</mu1>
-        <mu2>100000000000000.0</mu2>
-        <kp>1000000000000.0</kp>
-        <kd>10.0</kd>
-        <minDepth>0.001</minDepth>
-        <maxVel>10.0</maxVel>
-        <fdir1>1 0 0</fdir1>
     </gazebo>
-    <gazebo reference="left_wheel">
+    <gazebo reference="left_wheel_link">
         <material>Gazebo/Black</material>
-        <mu1>100000000000000.0</mu1>
-        <mu2>100000000000000.0</mu2>
-        <kp>1000000000000.0</kp>
-        <kd>10.0</kd>
-        <minDepth>0.001</minDepth>
-        <maxVel>10.0</maxVel>
-        <fdir1>1 0 0</fdir1>
     </gazebo>
-    <gazebo reference="base_caster_wheel">
+    <gazebo reference="caster_wheel_link">
         <material>Gazebo/Black</material>
         <mu1>0.1</mu1>
         <mu2>0.1</mu2>
-        <kp>1000000.0</kp>
-        <kd>100.0</kd>
-        <minDepth>0.001</minDepth>
-        <maxVel>10.0</maxVel>
     </gazebo>
     <gazebo>
@@ -51,5 +33,5 @@
             <robot_param>robot_description</robot_param>
             <robot_param_node>robot_state_publisher</robot_param_node>
-            <parameters>$(find axlr_controller)/config/axlr_controllers.yaml</parameters>
+            <!-- <parameters>$(find axlr_controller)/config/axlr_controllers.yaml</parameters> -->
         </plugin>
     </gazebo>

Commit message: fixed controller

File: src/axlr_description/urdf/axlr_core.urdf.xacro (robot description, xacro)
@@ -40,5 +40,5 @@
             <material name="black"/>
         </collision>
-        <xacro:cylinder_inertia m="0.5" r ="${wheel_diameter/2}" h="${wheel_length}"
+        <xacro:cylinder_inertia m="0.1" r ="${wheel_diameter/2}" h="${wheel_length}"
              xyz="0.0 0.0 0.0" rpy="0.0 0.0 0.0"/>
     </link>
@@ -64,5 +64,5 @@
             <material name="black"/>
         </collision>
-        <xacro:cylinder_inertia m="0.5" r ="${wheel_diameter/2}" h="${wheel_length}"
+        <xacro:cylinder_inertia m="0.1" r ="${wheel_diameter/2}" h="${wheel_length}"
              xyz="0.0 0.0 0.0" rpy="0.0 0.0 0.0"/>
     </link>
@@ -88,5 +88,5 @@
             <material name="black"/>
         </collision>
-        <xacro:sphere_inertia m="0.5" r ="${wheel_diameter/4}"
+        <xacro:sphere_inertia m="0.1" r ="${wheel_diameter/4}"
                 xyz="0.0 0.0 0.0" rpy="0.0 0.0 0.0"/>
     </link>

File: src/axlr_description/urdf/axlr_ros2_control.urdf.xacro (robot description, xacro)
@@ -1,8 +1,16 @@
 <?xml version="1.0"?>
 <robot xmlns:xacro="http://www.ros.org/wiki/xacro">
-    <ros2_control type="system" name="AXLR System">
+    <ros2_control name="GazeboSystem" type="system">
         <hardware>
             <plugin>gazebo_ros2_control/GazeboSystem</plugin>
         </hardware>
+        <joint name="left_wheel_joint">
+            <command_interface name="velocity">
+                <param name="min">-10</param>
+                <param name="max">10</param>
+            </command_interface>
+            <state_interface name="velocity"/>
+            <state_interface name="position"/>
+        </joint>
         <joint name="right_wheel_joint">
             <command_interface name="velocity">
@@ -10,14 +18,6 @@
                 <param name="max">10</param>
             </command_interface>
+            <state_interface name="velocity"/>
             <state_interface name="position"/>
-            <state_interface name="velocity"/>
-        </joint>
-        <joint name="left_wheel_joint">
-            <command_interface name="velocity">
-                <param name="min">-10</param>
-                <param name="max">10</param>
-            </command_interface>
-            <state_interface name="position"/>
-            <state_interface name="velocity"/>
         </joint>
     </ros2_control>

File: src/axlr_description/urdf/gazebo_properties.urdf.xacro (robot description, xacro)
@@ -1,38 +1,38 @@
 <?xml version="1.0"?>
-<robot xmlns:xacro="http://www.ros.org/wiki/xacro">
-    <transmission name="right_wheel_transmission">
-        <actuator name="right_wheel_motor" role="right_wheel_actuator"/>
-        <joint name="right_wheel_joint" role="right_joint">
-            <mechanicalReduction>1.0</mechanicalReduction>
-        </joint>
-        <plugin>transmission_interface/SimpleTransmission</plugin>
-    </transmission>
-    <transmission name="left_wheel_transmission">
-        <actuator name="left_wheel_motor" role="left_wheel_actuator"/>
-        <joint name="left_wheel_joint" role="left_joint">
-            <mechanicalReduction>1.0</mechanicalReduction>
-        </joint>
-        <plugin>transmission_interface/SimpleTransmission</plugin>
-    </transmission>
-    <gazebo reference="base_link">
-        <material>Gazebo/White</material>
-    </gazebo>
-    <gazebo reference="right_wheel_link">
-        <material>Gazebo/Black</material>
-    </gazebo>
-    <gazebo reference="left_wheel_link">
-        <material>Gazebo/Black</material>
-    </gazebo>
-    <gazebo reference="caster_wheel_link">
-        <material>Gazebo/Black</material>
-        <mu1>0.1</mu1>
-        <mu2>0.1</mu2>
-    </gazebo>
-    <gazebo>
-        <plugin filename="libgazebo_ros2_control.so" name="gazebo_ros2_control">
-            <robot_param>robot_description</robot_param>
-            <robot_param_node>robot_state_publisher</robot_param_node>
-            <parameters>$(find axlr_controller)/config/axlr_controllers.yaml</parameters>
-        </plugin>
-    </gazebo>
+<robot name="bumperbot" xmlns:xacro="http://ros.org/wiki/xacro">
+  <transmission name="wheel_right_transmission">
+    <plugin>transmission_interface/SimpleTransmission</plugin>
+    <actuator name="wheel_right_motor" role="actuator_right"/>
+    <joint name="right_wheel_joint"    role="joint_right">
+      <mechanical_reduction>1.0</mechanical_reduction>
+    </joint>
+  </transmission>
+  <transmission name="wheel_left_transmission">
+    <plugin>transmission_interface/SimpleTransmission</plugin>
+    <actuator name="wheel_left_motor" role="actuator_left"/>
+    <joint name="left_wheel_joint"    role="joint_left">
+      <mechanical_reduction>1.0</mechanical_reduction>
+    </joint>
+  </transmission>
+  <!-- Wheels -->
+  <gazebo reference="left_wheel">
+    <material>Gazebo/Blue</material>
+  </gazebo>
+  <gazebo reference="right_wheel">
+    <material>Gazebo/Blue</material>
+  </gazebo>
+  <!-- Caster Wheels -->
+  <gazebo reference="caster_wheel">
+    <material>Gazebo/Black</material>
+    <mu1>0.1</mu1>
+    <mu2>0.1</mu2>
+  </gazebo>
+  <!-- ROS 2 Control -->
+  <gazebo>
+    <plugin filename="libgazebo_ros2_control.so" name="gazebo_ros2_control">
+      <robot_param>robot_description</robot_param>
+      <robot_param_node>robot_state_publisher</robot_param_node>
+      <parameters>$(find axlr_controller)/config/axlr_controllers.yaml</parameters>
+    </plugin>
+  </gazebo>
 </robot>

File: src/axlr_description/urdf/main.urdf.xacro (robot description, xacro)
@@ -2,6 +2,6 @@
 <robot xmlns:xacro="http://www.ros.org/wiki/xacro" name="AXLR">
     <xacro:include filename="properties.urdf.xacro"/>
-    <xacro:include filename="inertial_macros.urdf.xacro"/>
-    <xacro:include filename="axlr_core.urdf.xacro"/>
+    <!-- <xacro:include filename="inertial_macros.urdf.xacro"/> -->
+    <xacro:include filename="core.urdf.xacro"/>
     <xacro:include filename="gazebo_properties.urdf.xacro"/>
     <xacro:include filename="axlr_ros2_control.urdf.xacro"/>
