Commit message: added odometry

File: src/axlr_description/urdf/axlr_ros2_control.urdf.xacro (robot description, xacro)
@@ -7,6 +7,6 @@
         <joint name="left_wheel_joint">
             <command_interface name="velocity">
-                <param name="min">-10</param>
-                <param name="max">10</param>
+                <param name="min">-1.0</param>
+                <param name="max">1.0</param>
             </command_interface>
             <state_interface name="velocity"/>
@@ -15,6 +15,6 @@
         <joint name="right_wheel_joint">
             <command_interface name="velocity">
-                <param name="min">-10</param>
-                <param name="max">10</param>
+                <param name="min">-1.0</param>
+                <param name="max">1.0</param>
             </command_interface>
             <state_interface name="velocity"/>

File: src/axlr_description/urdf/core.urdf.xacro (robot description, xacro)
@@ -61,6 +61,6 @@
         <parent link="base_link"/>
         <child link="left_wheel"/>
-        <origin xyz="0 0.17 0" rpy="-${pi/2} 0 0" />
-        <axis xyz="0 0 1"/>
+        <origin xyz="0 0.17 0" rpy="${pi/2} 0 0" />
+        <axis xyz="0 0 -1"/>
     </joint>
     <link name="left_wheel">

Commit message: continue later

File: src/axlr_description/urdf/axlr_ros2_control.urdf.xacro (robot description, xacro)
@@ -2,7 +2,15 @@
 <robot xmlns:xacro="http://www.ros.org/wiki/xacro">
     <ros2_control name="GazeboSystem" type="system">
-        <hardware>
-            <plugin>gazebo_ros2_control/GazeboSystem</plugin>
-        </hardware>
+        <xacro:if value="$(arg is_sim)">
+            <hardware>
+                <plugin>gazebo_ros2_control/GazeboSystem</plugin>
+            </hardware>
+        </xacro:if>
+        <xacro:unless value="$(arg is_sim)">
+            <hardware>
+                <plugin>axlr_firware/AXLRInterface</plugin>
+                <param name="port">/dev/ttyUSB0</param>
+            </hardware>
+        </xacro:unless>
         <joint name="left_wheel_joint">
             <command_interface name="velocity">

File: src/axlr_description/urdf/core.urdf.xacro (robot description, xacro)
@@ -1,4 +1,5 @@
 <?xml version="1.0"?>
 <robot xmlns:xacro="http://www.ros.org/wiki/xacro" >
+    <xacro:arg name="is_sim" default="true"/>
     <xacro:include filename="inertial_macro.urdf.xacro"/>
     <xacro:property name="chassis_width" value="0.266"/>

File: src/axlr_description/urdf/gazebo_properties.urdf.xacro (robot description, xacro)
@@ -28,4 +28,54 @@
     <mu2>0.1</mu2>
   </gazebo>
+  <gazebo reference="imu_link">
+      <material>Gazebo/Black</material>
+      <sensor name="imu" type="imu">
+        <always_on>true</always_on>
+        <update_rate>100</update_rate>
+        <imu>
+          <angular_velocity>
+            <x>
+              <noise type="gaussian">
+                <mean>0.0</mean>
+                <stddev>2e-4</stddev>
+              </noise>
+            </x>
+            <y>
+              <noise type="gaussian">
+                <mean>0.0</mean>
+                <stddev>2e-4</stddev>
+              </noise>
+            </y>
+            <z>
+              <noise type="gaussian">
+                <mean>0.0</mean>
+                <stddev>2e-4</stddev>
+              </noise>
+            </z>
+          </angular_velocity>
+          <linear_acceleration>
+            <x>
+              <noise type="gaussian">
+                <mean>0.0</mean>
+                <stddev>1.7e-2</stddev>
+              </noise>
+            </x>
+            <y>
+              <noise type="gaussian">
+                <mean>0.0</mean>
+                <stddev>1.7e-2</stddev>
+              </noise>
+            </y>
+            <z>
+              <noise type="gaussian">
+                <mean>0.0</mean>
+                <stddev>1.7e-2</stddev>
+              </noise>
+            </z>
+          </linear_acceleration>
+        </imu>
+        <plugin name="imu" filename="libgazebo_ros_imu_sensor.so"/>
+    </sensor>
+  </gazebo>
   <!-- ROS 2 Control -->
   <gazebo>

File: src/axlr_description/urdf/main.urdf.xacro (robot description, xacro)
@@ -4,4 +4,5 @@
     <!-- <xacro:include filename="inertial_macros.urdf.xacro"/> -->
     <xacro:include filename="core.urdf.xacro"/>
+    <xacro:include filename="imu.urdf.xacro"/>
     <xacro:include filename="gazebo_properties.urdf.xacro"/>
     <xacro:include filename="axlr_ros2_control.urdf.xacro"/>
